File: Kicad Fusée C'space/Kicad Fusée C'space.kicad_sch (KiCad schematic)
At the start: 9 parts, among them J1 Screw_Terminal_01x02, J2 Conn_01x02_Socket, J3 Conn_01x02_Socket, J4 Conn_01x02_Socket, J5 Conn_01x02_Socket, U2 BMP280, U3 MPU-6050

Commit message: programme V1
Parts:
- removed J4, J5: Conn_01x02_Socket, symbol Connector:Conn_01x02_Socket
- added D1: OK_LED, symbol Device:LED
- added D2: Err_LED, symbol Device:LED
- added D3: MBR3100RLG, symbol Device:D
- added F1: Fuse, symbol Device:Fuse
- added J6: Conn_01x02_Socket, symbol Connector:Conn_01x02_Socket
- added J7: Conn_02x08_Odd_Even, symbol Connector_Generic:Conn_02x08_Odd_Even
- added R1, R2: 470, symbol Device:R
- added R3, R4: R, symbol Device:R
- added R5: 1,7K, symbol Device:R
- added R6: 1,7k, symbol Device:R
- added U5: ~, symbol MyLib:BDX33B_
Connections:
- net +5V: now also U1.11 (V_{DD}), U1.32 (V_{DD}), D3.1 (K), F1.1, J7.5 (Pin_5), R2.1, R5.1, R6.1, U5.2 (C); no longer J1.1 (Pin_1)
- net GND: now also U1.12 (V_{SS}), U1.31 (V_{SS}), D1.1 (K), D2.1 (K), J6.2 (Pin_2), J7.1 (Pin_1), J7.15 (Pin_15)
- net SCKL: now also R5.2
- net SDA: now also R6.2
- net Fin course: now reaches U1.13 (RA7)
- net Fin course: now also J6.1 (Pin_1), R2.2
- net CS: now reaches U1.15 (RC0)
- net CS: now also J7.7 (Pin_7)
- net MOSI: now reaches U1.16 (RC1)
- net MOSI: now also J7.9 (Pin_9)
- net SCK: now reaches U1.17 (RC2)
- net SCK: now also J7.11 (Pin_11)
- net MISO: now reaches U1.18 (RC3)
- net MISO: now also J7.13 (Pin_13)
- net at U1.2 (RA0): now also R1.1
- net at U1.4 (RA2): now also R3.2
- net at U1.5 (RA3): now also R4.1
- net Motor OUT renamed Motor Output
- net Motor Output: now also D3.2 (A), U5.3 (E)
- new net: F1.2, J1.1 (Pin_1)
- new net: R1.2, U5.1 (B)
- new net: D2.2 (A), R4.2
- new net: D1.2 (A), R3.1
- no-connect marks 0 -> 46
Other:
- note added: "Alim"
- note added: "Capteur en I2C"
- note added: "Capteur pression atm"
- note added: "I2C pin et Pull Up resistance"
- note added: "Lecteur SD"
- note added: "Motor control"
- note added: "SD card info"
- note added: "SPI pin"
- note added: "fin course coiffe"
- moved on the sheet: J1, J2, J3, U2, U3, U4

Commit message: fin rce 3 sép timer
Other:
- note added: "raj timer en extern"
Changed lines of the file:
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@@
+    (effects (font (size 1.27 1.27)) (justify left bottom))
+  )
+  (text "raj timer en extern " (at 88.9 101.6 0)
     (effects (font (size 1.27 1.27)) (justify left bottom))
   )
